Commit message: Corrected package name

File: src/alpha/urdf/Alpha.xacro (robot description, xacro)
@@ -1,7 +1,7 @@
 <?xml version="1.0" ?>
 <robot name="Alpha" xmlns:xacro="http://www.ros.org/wiki/xacro">
-<xacro:include filename="$(find Alpha_description)/urdf/materials.xacro" />
-<xacro:include filename="$(find Alpha_description)/urdf/Alpha.trans" />
-<xacro:include filename="$(find Alpha_description)/urdf/Alpha.gazebo" />
+<xacro:include filename="$(find alpha)/urdf/materials.xacro" />
+<xacro:include filename="$(find alpha)/urdf/Alpha.trans" />
+<xacro:include filename="$(find alpha)/urdf/Alpha.gazebo" />
 <link name="base_link">
   <inertial>
@@ -13,5 +13,5 @@
     <origin rpy="0 0 0" xyz="0 0 0"/>
     <geometry>
-      <mesh filename="package://Alpha_description/meshes/base_link.stl" scale="0.001 0.001 0.001"/>
+      <mesh filename="package://alpha/meshes/base_link.stl" scale="0.001 0.001 0.001"/>
     </geometry>
     <material name="silver"/>
@@ -20,5 +20,5 @@
     <origin rpy="0 0 0" xyz="0 0 0"/>
     <geometry>
-      <mesh filename="package://Alpha_description/meshes/base_link.stl" scale="0.001 0.001 0.001"/>
+      <mesh filename="package://alpha/meshes/base_link.stl" scale="0.001 0.001 0.001"/>
     </geometry>
   </collision>
@@ -33,5 +33,5 @@
     <origin rpy="0 0 0" xyz="0.25 -0.33 -0.065"/>
     <geometry>
-      <mesh filename="package://Alpha_description/meshes/right_wheel_1.stl" scale="0.001 0.001 0.001"/>
+      <mesh filename="package://alpha/meshes/right_wheel_1.stl" scale="0.001 0.001 0.001"/>
     </geometry>
     <material name="silver"/>
@@ -40,5 +40,5 @@
     <origin rpy="0 0 0" xyz="0.25 -0.33 -0.065"/>
     <geometry>
-      <mesh filename="package://Alpha_description/meshes/right_wheel_1.stl" scale="0.001 0.001 0.001"/>
+      <mesh filename="package://alpha/meshes/right_wheel_1.stl" scale="0.001 0.001 0.001"/>
     </geometry>
   </collision>
@@ -53,5 +53,5 @@
     <origin rpy="0 0 0" xyz="-0.25 -0.33 -0.065"/>
     <geometry>
-      <mesh filename="package://Alpha_description/meshes/left_wheel_1.stl" scale="0.001 0.001 0.001"/>
+      <mesh filename="package://alpha/meshes/left_wheel_1.stl" scale="0.001 0.001 0.001"/>
     </geometry>
     <material name="silver"/>
@@ -60,5 +60,5 @@
     <origin rpy="0 0 0" xyz="-0.25 -0.33 -0.065"/>
     <geometry>
-      <mesh filename="package://Alpha_description/meshes/left_wheel_1.stl" scale="0.001 0.001 0.001"/>
+      <mesh filename="package://alpha/meshes/left_wheel_1.stl" scale="0.001 0.001 0.001"/>
     </geometry>
   </collision>
@@ -73,5 +73,5 @@
     <origin rpy="0 0 0" xyz="-0.0 -0.2 -0.015"/>
     <geometry>
-      <mesh filename="package://Alpha_description/meshes/caster_wheel_1.stl" scale="0.001 0.001 0.001"/>
+      <mesh filename="package://alpha/meshes/caster_wheel_1.stl" scale="0.001 0.001 0.001"/>
     </geometry>
     <material name="silver"/>
@@ -80,5 +80,5 @@
     <origin rpy="0 0 0" xyz="-0.0 -0.2 -0.015"/>
     <geometry>
-      <mesh filename="package://Alpha_description/meshes/caster_wheel_1.stl" scale="0.001 0.001 0.001"/>
+      <mesh filename="package://alpha/meshes/caster_wheel_1.stl" scale="0.001 0.001 0.001"/>
     </geometry>
   </collision>

Commit message: Differential Drive added

File: src/alpha/urdf/Alpha.xacro (robot description, xacro)
@@ -88,5 +88,5 @@
   <parent link="base_link"/>
   <child link="right_wheel_1"/>
-  <axis xyz="-1.0 0.0 0.0"/>
+  <axis xyz="1 0 0"/>
 </joint>
 <joint name="Rev2" type="continuous">
@@ -94,5 +94,5 @@
   <parent link="base_link"/>
   <child link="left_wheel_1"/>
-  <axis xyz="1.0 0.0 0.0"/>
+  <axis xyz="1 0 0"/>
 </joint>
 <joint name="Rigid3" type="fixed">
