Commit message: Visual and differential drive plugin added

File: src/beta_description/urdf/beta.xacro (robot description, xacro)
@@ -148,5 +148,5 @@
   <parent link="base_link"/>
   <child link="left_wheel_1"/>
-  <axis xyz="0.0 -1.0 0.0"/>
+  <axis xyz="0.0 1.0 0.0"/>
 </joint>
 <joint name="right_whell_joint" type="continuous">
@@ -154,5 +154,5 @@
   <parent link="base_link"/>
   <child link="right_wheel_1"/>
-  <axis xyz="0.0 -1.0 0.0"/>
+  <axis xyz="0.0 1.0 0.0"/>
 </joint>
 <joint name="lidar_joint" type="fixed">

Commit message: Camera Added

File: src/beta_description/urdf/beta.xacro (robot description, xacro)
@@ -84,5 +84,5 @@
   </collision>
 </link>
-<link name="camera_link_1">
+<link name="camera">
   <inertial>
     <origin rpy="0 0 0" xyz="0.004999999999999977 0.0 0.0"/>
@@ -164,5 +164,5 @@
   <origin rpy="0 0 0" xyz="0.15 0.0 0.05"/>
   <parent link="base_link"/>
-  <child link="camera_link_1"/>
+  <child link="camera"/>
 </joint>
 <joint name="pi_joint" type="fixed">

Commit message: LiDAR added and TF published

File: src/beta_description/urdf/beta.xacro (robot description, xacro)
@@ -67,9 +67,9 @@
   <inertial>
     <origin rpy="0 0 0" xyz="-0.03 -0.06999999999999999 0.007500000000000007"/>
-    <mass value="0.011925"/>
+    <mass value="1e-5"/>
     <inertia ixx="1e-06" ixy="-0.0" ixz="0.0" iyy="1e-06" iyz="0.0" izz="2e-06"/>
   </inertial>
   <visual>
-    <origin rpy="0 0 0" xyz="-0.15 -0.075 -0.075"/>
+    <origin rpy="0 0 0" xyz="-0.15 -0.0 -0.09"/>
     <geometry>
       <mesh filename="package://beta_description/meshes/lidar_link_1.stl" scale="0.001 0.001 0.001"/>
@@ -78,5 +78,5 @@
   </visual>
   <collision>
-    <origin rpy="0 0 0" xyz="-0.15 -0.075 -0.075"/>
+    <origin rpy="0 0 0" xyz="-0.15 -0.0 -0.09"/>
     <geometry>
       <mesh filename="package://beta_description/meshes/lidar_link_1.stl" scale="0.001 0.001 0.001"/>
@@ -157,5 +157,6 @@
 </joint>
 <joint name="lidar_joint" type="fixed">
-  <origin rpy="0 0 0" xyz="0.15 0.075 0.075"/>
+  <!--<origin rpy="0 0 0" xyz="0.15 0 0.075"/> -->
+  <origin rpy="0 0 0" xyz="0.15 0 0.09"/>
   <parent link="base_link"/>
   <child link="lidar_link_1"/>
